Commit message: comments fix

File: src/rover_description/urdf/oakd.xacro (robot description, xacro)
@@ -6,5 +6,5 @@
   <xacro:property name="oakd_right_offset" value="0 -0.375 0"/>
   <xacro:property name="oakd_mesh" value="package://rover_description/meshes/oak_d.dae"/>
-  <!-- Kamery stereo -->
+  <!-- Stereo Cameras -->
   <xacro:macro name="oakd_stereo_camera" params="name parent_link offset frame_id topic camera_info_topic joint_name">
     <link name="${name}"/>
@@ -39,5 +39,5 @@
     </gazebo>
   </xacro:macro>
-  <!-- Lewa kamera stereo -->
+  <!-- Left Stereo Camera -->
   <xacro:oakd_stereo_camera
     name="oakd_camera_left"
@@ -47,5 +47,5 @@
     topic="/stereo/left/image_raw"
     camera_info_topic="/stereo/left/camera_info"/>
-  <!-- Prawa kamera stereo -->
+  <!-- Right Stereo Camera -->
   <xacro:oakd_stereo_camera
     name="oakd_camera_right"
@@ -55,5 +55,5 @@
     topic="/stereo/right/image_raw"
     camera_info_topic="/stereo/right/camera_info"/>
-  <!-- Makro dla sensora depth_camera (depth lub pointcloud) -->
+  <!-- Depth Camera Sensor (depth or pointcloud) -->
   <xacro:macro name="oakd_depth_sensor" params="name topic camera_info_topic frame_id output_type">
     <gazebo reference="oakd_camera_center">
@@ -88,8 +88,9 @@
         </camera>
         <frame_id>${frame_id}</frame_id>
-      </sensor>
-    </gazebo>
-  </xacro:macro>
-  <!-- Makro dla RGB camera -->
+        <gz_frame_id>${frame_id}</gz_frame_id>
+      </sensor>
+    </gazebo>
+  </xacro:macro>
+  <!-- RGB Camera Sensor -->
   <xacro:macro name="oakd_rgb_sensor" params="name topic camera_info_topic frame_id">
     <gazebo reference="oakd_camera_center">
@@ -121,5 +122,5 @@
     </gazebo>
   </xacro:macro>
-  <!-- Makro dla IMU -->
+  <!-- IMU Sensor -->
   <xacro:macro name="oakd_imu_sensor" params="name topic frame_id">
     <gazebo reference="oakd_camera_center">
@@ -134,7 +135,6 @@
     </gazebo>
   </xacro:macro>
-  <!-- Główne makro modułu OAK-D -->
   <xacro:macro name="oakd_module" params="parent_link:=base_link">
-    <!-- Główny korpus OAK-D -->
+    <!-- OAK-D Core -->
     <link name="oakd_camera_center">
       <visual>
@@ -154,5 +154,5 @@
       </inertial>
     </link>
-    <!-- Joint do bazy (parametryzowany) -->
+    <!-- Joint to base (parameterized) -->
     <joint name="oakd_camera_link" type="fixed">
       <parent link="${parent_link}" />
@@ -160,5 +160,12 @@
       <origin xyz="${oakd_center_xyz}" rpy="0 0 0" />
     </joint>
-    <!-- Lewa kamera stereo -->
+    <!-- Optical frame: X to the right, Y down, Z forward -->
+    <link name="oakd_camera_optical_frame"/>
+    <joint name="oakd_camera_optical_joint" type="fixed">
+      <parent link="oakd_camera_center" />
+      <child link="oakd_camera_optical_frame" />
+      <origin xyz="0 0 0" rpy="-1.5708 0 -1.5708" />
+    </joint>
+    <!-- Left Stereo Camera -->
     <xacro:oakd_stereo_camera
       name="oakd_camera_left"
@@ -169,5 +176,5 @@
       camera_info_topic="/stereo/left/camera_info"
       joint_name="oakd_left_camera_joint"/>
-    <!-- Prawa kamera stereo -->
+    <!-- Right Stereo Camera -->
     <xacro:oakd_stereo_camera
       name="oakd_camera_right"
@@ -183,5 +190,5 @@
       topic="/depth/image_raw"
       camera_info_topic="/depth/camera_info"
-      frame_id="oakd_camera_center"
+      frame_id="oakd_camera_optical_frame"
       output_type="depth"/>
     <!-- PointCloud2 -->
@@ -190,5 +197,5 @@
       topic="/points"
       camera_info_topic=""
-      frame_id="oakd_camera_center"
+      frame_id="oakd_camera_optical_frame"
       output_type="pointcloud"/>
     <!-- RGB camera -->
