Commit message: oak-d vision works

File: src/rover_description/urdf/rex.urdf (robot description, URDF)
Before this commit: robot rex, 24 links, 23 joints
Links:
- added link oakd_camera_link, mass 0.2; collision box size=0.08 0.03 0.03; visual box size=0.08 0.03 0.03
Joints:
- added joint oakd_camera_joint: type fixed, parent base_link, child oakd_camera_link, origin xyz=0.38 0 0.10 rpy=0 0 0

Commit message: Some oakd parameters fixed

File: src/rover_description/urdf/rex.urdf (robot description, URDF)
Before this commit: robot rex, 25 links, 24 joints
Links:
- removed link oakd_camera_link
- added link oakd_camera, mass 0.1; collision mesh filename=package://rover_description/meshes/oak_d.dae; visual mesh filename=package://rover_description/meshes/oak_d.dae
Joints:
- removed joint oakd_camera_joint
- added joint oakd_camera_link: type fixed, parent base_link, child oakd_camera, origin xyz=0.38 0 0.10 rpy=0 0 0

Commit message: camera position fixed

File: src/rover_description/urdf/rex.urdf (robot description, URDF)
Before this commit: robot rex, 25 links, 24 joints
Links:
- removed link oakd_camera
- added link oakd_camera_center, mass 0.1; collision mesh filename=package://rover_description/meshes/oak_d.dae; visual mesh filename=package://rover_description/meshes/oak_d.dae
- added link oakd_camera_left
- added link oakd_camera_right
Joints:
- added joint oakd_left_camera_joint: type fixed, parent oakd_camera_center, child oakd_camera_left, origin xyz=0 0.375 0 rpy=0 0 0
- added joint oakd_right_camera_joint: type fixed, parent oakd_camera_center, child oakd_camera_right, origin xyz=0 -0.375 0 rpy=0 0 0
- joint oakd_camera_link: child oakd_camera -> oakd_camera_center

Commit message: bridge fixed and rviz cloud working

File: src/rover_description/urdf/rex.urdf (robot description, URDF)
Before this commit: robot rex, 27 links, 26 joints
Links:
- added link oakd_camera_optical_frame
Joints:
- added joint oakd_camera_optical_joint: type fixed, parent oakd_camera_center, child oakd_camera_optical_frame, origin xyz=0 0 0 rpy=-1.5708 0 -1.5708

Commit message: oakd pro added to rex.urdf

File: src/rover_description/urdf/rex.urdf (robot description, URDF)
Before this commit: robot rex, 28 links, 27 joints
Links:
- added link oakd_pro_camera_center, mass 0.09; collision mesh filename=package://rover_description/meshes/oak_d_pro.dae; visual mesh filename=package://rover_description/meshes/oak_d_pro.dae
- added link oakd_pro_camera_left
- added link oakd_pro_camera_optical_frame
- added link oakd_pro_camera_right
Joints:
- added joint oakd_pro_camera_link: type fixed, parent base_link, child oakd_pro_camera_center, origin xyz=0.38 0 0.20 rpy=0 0 0
- added joint oakd_pro_camera_optical_joint: type fixed, parent oakd_pro_camera_center, child oakd_pro_camera_optical_frame, origin xyz=0 0 0 rpy=-1.5708 0 -1.5708
- added joint oakd_pro_left_camera_joint: type fixed, parent oakd_pro_camera_center, child oakd_pro_camera_left, origin xyz=0 0.375 0 rpy=0 0 0
- added joint oakd_pro_right_camera_joint: type fixed, parent oakd_pro_camera_center, child oakd_pro_camera_right, origin xyz=0 -0.375 0 rpy=0 0 0

Commit message: oakd pro in different file

File: src/rover_description/urdf/rex.urdf (robot description, URDF)
Before this commit: robot rex, 32 links, 31 joints
Links:
- removed link oakd_pro_camera_center
- removed link oakd_pro_camera_left
- removed link oakd_pro_camera_optical_frame
- removed link oakd_pro_camera_right
Joints:
- removed joint oakd_pro_camera_link
- removed joint oakd_pro_camera_optical_joint
- removed joint oakd_pro_left_camera_joint
- removed joint oakd_pro_right_camera_joint

Commit message: bridge configured for oakd pro and fixes in oakd pro urdf

File: src/rover_description/urdf/rex.urdf (robot description, URDF)
Before this commit: robot rex, 28 links, 27 joints
Links:
- removed link oakd_camera_center
- removed link oakd_camera_left
- removed link oakd_camera_optical_frame
- removed link oakd_camera_right
- added link oakd_pro_camera_center, mass 0.09; collision mesh filename=package://rover_description/meshes/oak_d_pro_w.dae scale=0.001 0.001 0.001; visual mesh filename=package://rover_description/meshes/oak_d_pro_w.dae scale=0.001 0.001 0.001
- added link oakd_pro_camera_left
- added link oakd_pro_camera_optical_frame
- added link oakd_pro_camera_right
Joints:
- removed joint oakd_camera_link
- removed joint oakd_camera_optical_joint
- removed joint oakd_left_camera_joint
- removed joint oakd_right_camera_joint
- added joint oakd_pro_camera_link: type fixed, parent base_link, child oakd_pro_camera_center, origin xyz=0.38 0.04 0.10 rpy=0 0 0
- added joint oakd_pro_camera_optical_joint: type fixed, parent oakd_pro_camera_center, child oakd_pro_camera_optical_frame, origin xyz=0 0 0 rpy=-1.5708 0 -1.5708
- added joint oakd_pro_left_camera_joint: type fixed, parent oakd_pro_camera_center, child oakd_pro_camera_left, origin xyz=0 0.375 0 rpy=0 0 0
- added joint oakd_pro_right_camera_joint: type fixed, parent oakd_pro_camera_center, child oakd_pro_camera_right, origin xyz=0 -0.375 0 rpy=0 0 0
