Commit message: Aktualizacja nav2 i dodanie skryptu obrotu

File: src/rover_description/urdf/rex.urdf (robot description, URDF)
Before this commit: robot rex, 28 links, 27 joints
Joints:
- joint base_link_to_swivel_left: limit lower=-1 upper=1 effort=1000.0 velocity=0.5 -> lower=-1 upper=1 effort=1000.0 velocity=5.0
- joint base_link_to_swivel_right: limit lower=-1 upper=1 effort=1000.0 velocity=0.5 -> lower=-1 upper=1 effort=1000.0 velocity=5.0
- joint motor_front_left_to_steer_front_left: limit lower=-3.14159265 upper=3.14159265 effort=10.0 velocity=0.76 -> lower=-3.14159265 upper=3.14159265 effort=10.0 velocity=5.0
- joint motor_front_right_to_steer_front_right: limit lower=-3.14159265 upper=3.14159265 effort=10.0 velocity=0.76 -> lower=-3.14159265 upper=3.14159265 effort=10.0 velocity=5.0
- joint motor_rear_left_to_steer_rear_left: limit lower=-3.14159265 upper=3.14159265 effort=10.0 velocity=0.76 -> lower=-3.14159265 upper=3.14159265 effort=10.0 velocity=5.0
- joint motor_rear_right_to_steer_rear_right: limit lower=-3.14159265 upper=3.14159265 effort=10.0 velocity=0.76 -> lower=-3.14159265 upper=3.14159265 effort=10.0 velocity=5.0

File: src/rover_description/urdf/rex_donot_touch.urdf (robot description, URDF)
Before this commit: robot rex, 17 links, 16 joints
Joints:
- joint base_link_to_swivel_left: limit lower=-1 upper=1 effort=1000.0 velocity=0.5 -> lower=-1 upper=1 effort=1000.0 velocity=5.0
- joint base_link_to_swivel_right: limit lower=-1 upper=1 effort=1000.0 velocity=0.5 -> lower=-1 upper=1 effort=1000.0 velocity=5.0
- joint motor_front_left_to_steer_front_left: limit lower=-3.14159265 upper=3.14159265 effort=10.0 velocity=0.76 -> lower=-3.14159265 upper=3.14159265 effort=10.0 velocity=5.0
- joint motor_front_right_to_steer_front_right: limit lower=-3.14159265 upper=3.14159265 effort=10.0 velocity=0.76 -> lower=-3.14159265 upper=3.14159265 effort=10.0 velocity=5.0
- joint motor_rear_left_to_steer_rear_left: limit lower=-3.14159265 upper=3.14159265 effort=10.0 velocity=0.76 -> lower=-3.14159265 upper=3.14159265 effort=10.0 velocity=5.0
- joint motor_rear_right_to_steer_rear_right: limit lower=-3.14159265 upper=3.14159265 effort=10.0 velocity=0.76 -> lower=-3.14159265 upper=3.14159265 effort=10.0 velocity=5.0

File: src/rover_description/urdf/xacro/wheel_assembly.xacro (robot description, xacro)
@@ -10,5 +10,5 @@
       <origin xyz="${x} 0 -0.05" rpy="0 0 0"/>
       <axis xyz="0 0 1"/>
-      <limit effort="10.0" lower="-3.14159265" upper="3.14159265" velocity="0.76"/>
+      <limit effort="10.0" lower="-3.14159265" upper="3.14159265" velocity="5.0"/>
     </joint>
     <!-- Steering shaft -->
@@ -95,5 +95,5 @@
       <origin xyz="0 ${base_y} 0" rpy="0 0 0"/>
       <axis xyz="0 1 0"/>
-      <limit effort="1000.0" lower="-1.15" upper="1.15" velocity="0.6"/>
+      <limit effort="1000.0" lower="-1.15" upper="1.15" velocity="5.0"/>
       <dynamics friction="1.0" damping="0.1"/>
     </joint>
@@ -158,5 +158,5 @@
       <origin xyz="0.05 0 0" rpy="0 0 0"/>
       <axis xyz="0 1 0"/>
-      <limit effort="500.0" lower="-0.7" upper="0.7" velocity="0.6"/>
+      <limit effort="500.0" lower="-0.7" upper="0.7" velocity="5.0"/>
       <dynamics friction="0.3" damping="0.05"/>
     </joint>
@@ -191,5 +191,5 @@
       <origin xyz="-0.05 0 0" rpy="0 0 0"/>
       <axis xyz="0 1 0"/>
-      <limit effort="500.0" lower="-0.7" upper="0.7" velocity="0.6"/>
+      <limit effort="500.0" lower="-0.7" upper="0.7" velocity="5.0"/>
       <dynamics friction="0.3" damping="0.05"/>
     </joint>

Commit message: Revert URDF velocity limit changes

File: src/rover_description/urdf/rex.urdf (robot description, URDF)
Before this commit: robot rex, 28 links, 27 joints
Joints:
- joint base_link_to_swivel_left: limit lower=-1 upper=1 effort=1000.0 velocity=5.0 -> lower=-1 upper=1 effort=1000.0 velocity=0.5
- joint base_link_to_swivel_right: limit lower=-1 upper=1 effort=1000.0 velocity=5.0 -> lower=-1 upper=1 effort=1000.0 velocity=0.5
- joint motor_front_left_to_steer_front_left: limit lower=-3.14159265 upper=3.14159265 effort=10.0 velocity=5.0 -> lower=-3.14159265 upper=3.14159265 effort=10.0 velocity=0.76
- joint motor_front_right_to_steer_front_right: limit lower=-3.14159265 upper=3.14159265 effort=10.0 velocity=5.0 -> lower=-3.14159265 upper=3.14159265 effort=10.0 velocity=0.76
- joint motor_rear_left_to_steer_rear_left: limit lower=-3.14159265 upper=3.14159265 effort=10.0 velocity=5.0 -> lower=-3.14159265 upper=3.14159265 effort=10.0 velocity=0.76
- joint motor_rear_right_to_steer_rear_right: limit lower=-3.14159265 upper=3.14159265 effort=10.0 velocity=5.0 -> lower=-3.14159265 upper=3.14159265 effort=10.0 velocity=0.76

File: src/rover_description/urdf/rex_donot_touch.urdf (robot description, URDF)
Before this commit: robot rex, 17 links, 16 joints
Joints:
- joint base_link_to_swivel_left: limit lower=-1 upper=1 effort=1000.0 velocity=5.0 -> lower=-1 upper=1 effort=1000.0 velocity=0.5
- joint base_link_to_swivel_right: limit lower=-1 upper=1 effort=1000.0 velocity=5.0 -> lower=-1 upper=1 effort=1000.0 velocity=0.5
- joint motor_front_left_to_steer_front_left: limit lower=-3.14159265 upper=3.14159265 effort=10.0 velocity=5.0 -> lower=-3.14159265 upper=3.14159265 effort=10.0 velocity=0.76
- joint motor_front_right_to_steer_front_right: limit lower=-3.14159265 upper=3.14159265 effort=10.0 velocity=5.0 -> lower=-3.14159265 upper=3.14159265 effort=10.0 velocity=0.76
- joint motor_rear_left_to_steer_rear_left: limit lower=-3.14159265 upper=3.14159265 effort=10.0 velocity=5.0 -> lower=-3.14159265 upper=3.14159265 effort=10.0 velocity=0.76
- joint motor_rear_right_to_steer_rear_right: limit lower=-3.14159265 upper=3.14159265 effort=10.0 velocity=5.0 -> lower=-3.14159265 upper=3.14159265 effort=10.0 velocity=0.76

File: src/rover_description/urdf/xacro/wheel_assembly.xacro (robot description, xacro)
@@ -10,5 +10,5 @@
       <origin xyz="${x} 0 -0.05" rpy="0 0 0"/>
       <axis xyz="0 0 1"/>
-      <limit effort="10.0" lower="-3.14159265" upper="3.14159265" velocity="5.0"/>
+      <limit effort="10.0" lower="-3.14159265" upper="3.14159265" velocity="0.76"/>
     </joint>
     <!-- Steering shaft -->
@@ -95,5 +95,5 @@
       <origin xyz="0 ${base_y} 0" rpy="0 0 0"/>
       <axis xyz="0 1 0"/>
-      <limit effort="1000.0" lower="-1.15" upper="1.15" velocity="5.0"/>
+      <limit effort="1000.0" lower="-1.15" upper="1.15" velocity="0.6"/>
       <dynamics friction="1.0" damping="0.1"/>
     </joint>
@@ -158,5 +158,5 @@
       <origin xyz="0.05 0 0" rpy="0 0 0"/>
       <axis xyz="0 1 0"/>
-      <limit effort="500.0" lower="-0.7" upper="0.7" velocity="5.0"/>
+      <limit effort="500.0" lower="-0.7" upper="0.7" velocity="0.6"/>
       <dynamics friction="0.3" damping="0.05"/>
     </joint>
@@ -191,5 +191,5 @@
       <origin xyz="-0.05 0 0" rpy="0 0 0"/>
       <axis xyz="0 1 0"/>
-      <limit effort="500.0" lower="-0.7" upper="0.7" velocity="5.0"/>
+      <limit effort="500.0" lower="-0.7" upper="0.7" velocity="0.6"/>
       <dynamics friction="0.3" damping="0.05"/>
     </joint>
