Commit message: oakd pro xacro created and oakd xacro fixed

File: src/rover_description/urdf/oakd_pro.xacro (robot description, xacro)
@@ -1,11 +1,17 @@
 <?xml version="1.0"?>
-<robot name="oakd" xmlns:xacro="http://ros.org/wiki/xacro">
+<robot name="oakd_pro" xmlns:xacro="http://ros.org/wiki/xacro">
   <!-- Parametry konfiguracyjne -->
-  <xacro:property name="oakd_center_xyz" value="0.38 0 0.10"/>
-  <xacro:property name="oakd_left_offset" value="0 0.375 0"/>
-  <xacro:property name="oakd_right_offset" value="0 -0.375 0"/>
-  <xacro:property name="oakd_mesh" value="package://rover_description/meshes/oak_d.dae"/>
+  <xacro:property name="oakd_pro_center_xyz" value="0.38 0.04 0.10"/>
+  <xacro:property name="oakd_pro_left_offset" value="0 0.375 0"/>
+  <xacro:property name="oakd_pro_right_offset" value="0 -0.375 0"/>
+  <xacro:property name="oakd_pro_mesh" value="package://rover_description/meshes/oak_d_pro_w.dae"/>
+  <xacro:property name="oakd_pro_mesh_scale" value="0.001 0.001 0.001"/>
+  <!--
+    oak_d_pro_w.dae has Y_UP, while the rest of the robot is Z_UP.
+    This rpy rotates the mesh to match the robot/Gazebo convention.
+  -->
+  <xacro:property name="oakd_pro_mesh_rpy" value="1.5708 0 -1.5708"/>
   <!-- Stereo Cameras -->
-  <xacro:macro name="oakd_stereo_camera" params="name parent_link offset frame_id topic camera_info_topic joint_name">
+  <xacro:macro name="oakd_pro_stereo_camera" params="name parent_link offset frame_id topic camera_info_topic joint_name">
     <link name="${name}"/>
     <joint name="${joint_name}" type="fixed">
@@ -24,5 +30,5 @@
             <camera_info_topic>${camera_info_topic}</camera_info_topic>
           </xacro:if>
-          <horizontal_fov>1.25663</horizontal_fov>
+          <horizontal_fov>1.39626</horizontal_fov>
           <image>
             <width>640</width>
@@ -40,6 +46,6 @@
   </xacro:macro>
   <!-- Depth Camera Sensor (depth or pointcloud) -->
-  <xacro:macro name="oakd_depth_sensor" params="name topic camera_info_topic frame_id output_type">
-    <gazebo reference="oakd_camera_center">
+  <xacro:macro name="oakd_pro_depth_sensor" params="name topic camera_info_topic frame_id output_type">
+    <gazebo reference="oakd_pro_camera_center">
       <sensor name="${name}" type="depth_camera">
         <always_on>true</always_on>
@@ -48,6 +54,8 @@
         <topic>${topic}</topic>
         <camera name="${name}_camera">
-          <camera_info_topic>${camera_info_topic}</camera_info_topic>
-          <horizontal_fov>1.25663</horizontal_fov>
+          <xacro:if value="${camera_info_topic != ''}">
+            <camera_info_topic>${camera_info_topic}</camera_info_topic>
+          </xacro:if>
+          <horizontal_fov>1.39626</horizontal_fov>
           <image>
             <width>640</width>
@@ -77,6 +85,6 @@
   </xacro:macro>
   <!-- RGB Camera Sensor -->
-  <xacro:macro name="oakd_rgb_sensor" params="name topic camera_info_topic frame_id">
-    <gazebo reference="oakd_camera_center">
+  <xacro:macro name="oakd_pro_rgb_sensor" params="name topic camera_info_topic frame_id">
+    <gazebo reference="oakd_pro_camera_center">
       <sensor name="${name}" type="camera">
         <always_on>true</always_on>
@@ -86,5 +94,5 @@
         <camera name="${name}_camera">
           <camera_info_topic>${camera_info_topic}</camera_info_topic>
-          <horizontal_fov>1.20427</horizontal_fov>
+          <horizontal_fov>1.15191</horizontal_fov>
           <image>
             <width>1280</width>
@@ -107,6 +115,6 @@
   </xacro:macro>
   <!-- IMU Sensor -->
-  <xacro:macro name="oakd_imu_sensor" params="name topic frame_id">
-    <gazebo reference="oakd_camera_center">
+  <xacro:macro name="oakd_pro_imu_sensor" params="name topic frame_id">
+    <gazebo reference="oakd_pro_camera_center">
       <sensor name="${name}" type="imu">
         <always_on>1</always_on>
@@ -119,79 +127,81 @@
     </gazebo>
   </xacro:macro>
-  <xacro:macro name="oakd_module" params="parent_link:=base_link">
-    <!-- OAK-D Core -->
-    <link name="oakd_camera_center">
+  <xacro:macro name="oakd_pro_module" params="parent_link:=base_link">
+    <!-- OAK-D Pro W Core -->
+    <link name="oakd_pro_camera_center">
       <visual>
+        <origin xyz="0 0 0" rpy="${oakd_pro_mesh_rpy}" />
         <geometry>
-          <mesh filename="${oakd_mesh}"/>
+          <mesh filename="${oakd_pro_mesh}" scale="${oakd_pro_mesh_scale}"/>
         </geometry>
       </visual>
       <collision>
+        <origin xyz="0 0 0" rpy="${oakd_pro_mesh_rpy}" />
         <geometry>
-          <mesh filename="${oakd_mesh}"/>
+          <mesh filename="${oakd_pro_mesh}" scale="${oakd_pro_mesh_scale}"/>
         </geometry>
       </collision>
       <inertial>
         <origin xyz="0 0 0" />
-        <mass value="0.1" />
+        <mass value="0.09" />
         <inertia ixx="0.0001" ixy="0" ixz="0" iyy="0.0001" iyz="0" izz="0.0001" />
       </inertial>
     </link>
     <!-- Joint to base (parameterized) -->
-    <joint name="oakd_camera_link" type="fixed">
+    <joint name="oakd_pro_camera_link" type="fixed">
       <parent link="${parent_link}" />
-      <child link="oakd_camera_center" />
-      <origin xyz="${oakd_center_xyz}" rpy="0 0 0" />
+      <child link="oakd_pro_camera_center" />
+      <origin xyz="${oakd_pro_center_xyz}" rpy="0 0 0" />
     </joint>
     <!-- Optical frame: X to the right, Y down, Z forward -->
-    <link name="oakd_camera_optical_frame"/>
-    <joint name="oakd_camera_optical_joint" type="fixed">
-      <parent link="oakd_camera_center" />
-      <child link="oakd_camera_optical_frame" />
+    <link name="oakd_pro_camera_optical_frame"/>
+    <joint name="oakd_pro_camera_optical_joint" type="fixed">
+      <parent link="oakd_pro_camera_center" />
+      <child link="oakd_pro_camera_optical_frame" />
       <origin xyz="0 0 0" rpy="-1.5708 0 -1.5708" />
     </joint>
     <!-- Left Stereo Camera -->
-    <xacro:oakd_stereo_camera
-      name="oakd_camera_left"
-      parent_link="oakd_camera_center"
-      offset="${oakd_left_offset}"
-      frame_id="oakd_camera_left"
+    <xacro:oakd_pro_stereo_camera
+      name="oakd_pro_camera_left"
+      parent_link="oakd_pro_camera_center"
+      offset="${oakd_pro_left_offset}"
+      frame_id="oakd_pro_camera_left"
       topic="/stereo/left/image_raw"
       camera_info_topic="/stereo/left/camera_info"
-      joint_name="oakd_left_camera_joint"/>
+      joint_name="oakd_pro_left_camera_joint"/>
     <!-- Right Stereo Camera -->
-    <xacro:oakd_stereo_camera
-      name="oakd_camera_right"
-      parent_link="oakd_camera_center"
-      offset="${oakd_right_offset}"
-      frame_id="oakd_camera_right"
+    <xacro:oakd_pro_stereo_camera
+      name="oakd_pro_camera_right"
+      parent_link="oakd_pro_camera_center"
+      offset="${oakd_pro_right_offset}"
+      frame_id="oakd_pro_camera_right"
       topic="/stereo/right/image_raw"
       camera_info_topic="/stereo/right/camera_info"
-      joint_name="oakd_right_camera_joint"/>
+      joint_name="oakd_pro_right_camera_joint"/>
     <!-- Depth (image) -->
-    <xacro:oakd_depth_sensor
-      name="oakd_depth"
+    <xacro:oakd_pro_depth_sensor
+      name="oakd_pro_depth"
       topic="/depth/image_raw"
       camera_info_topic="/depth/camera_info"
-      frame_id="oakd_camera_optical_frame"
+      frame_id="oakd_pro_camera_optical_frame"
       output_type="depth"/>
     <!-- PointCloud2 -->
-    <xacro:oakd_depth_sensor
-      name="oakd_points"
+    <xacro:oakd_pro_depth_sensor
+      name="oakd_pro_points"
       topic="/points"
       camera_info_topic=""
-      frame_id="oakd_camera_optical_frame"
+      frame_id="oakd_pro_camera_optical_frame"
       output_type="pointcloud"/>
     <!-- RGB camera -->
-    <xacro:oakd_rgb_sensor
-      name="oakd_rgb"
+    <xacro:oakd_pro_rgb_sensor
+      name="oakd_pro_rgb"
       topic="/rgb/image_raw"
       camera_info_topic="/rgb/camera_info"
-      frame_id="oakd_camera_center"/>
+      frame_id="oakd_pro_camera_center"/>
     <!-- IMU -->
-    <xacro:oakd_imu_sensor
-      name="oakd_imu"
+    <xacro:oakd_pro_imu_sensor
+      name="oakd_pro_imu"
       topic="/imu/data"
-      frame_id="oakd_camera_center"/>
+      frame_id="oakd_pro_camera_center"/>
   </xacro:macro>
 </robot>
