Commit message: refactor: migrate OAK-D camera sensors to reusable xacro macros

File: src/rover_description/urdf/rex.urdf.xacro (robot description, xacro)
@@ -13,3 +13,13 @@
   <!-- Gazebo plugins -->
   <xacro:gazebo_plugins/>
+  <!-- <xacro:include filename="$(find rover_description)/urdf/xacro/macros/camera_assembly.xacro"/>
+  <xacro:camera_assembly parent_link="base_link" camera_center_xyz="0.40 0.0 0.10"/> -->
+  <xacro:include filename="$(find rover_description)/urdf/xacro/macros/oak_d_camera_assembly.xacro"/>
+  <xacro:oak_d_camera name="camera" parent_link="base_link">
+    <origin xyz="0.40 0.0 0.10" rpy="0 0 0" />
+  </xacro:oak_d_camera>
+  <!-- <xacro:include filename="$(find rover_description)/urdf/xacro/oakd.xacro"/>
+  <xacro:include filename="$(find rover_description)/urdf/xacro/oakd_pro.xacro"/> -->
+  <!-- <xacro:oakd_module parent_link="base_link"/> -->
+  <!-- <xacro:oakd_pro_module parent_link="base_link"/> -->
 </robot>

Commit message: feat: integrate Ouster OS1 lidar and refactor sensor assemblies

File: src/rover_description/urdf/rex.urdf.xacro (robot description, xacro)
@@ -13,13 +13,11 @@
   <!-- Gazebo plugins -->
   <xacro:gazebo_plugins/>
-  <!-- <xacro:include filename="$(find rover_description)/urdf/xacro/macros/camera_assembly.xacro"/>
-  <xacro:camera_assembly parent_link="base_link" camera_center_xyz="0.40 0.0 0.10"/> -->
-  <xacro:include filename="$(find rover_description)/urdf/xacro/macros/oak_d_camera_assembly.xacro"/>
-  <xacro:oak_d_camera name="camera" parent_link="base_link">
+  <!-- <xacro:include filename="$(find rover_description)/urdf/xacro/macros/oak_d_pro_w_camera_assembly.xacro"/>
+  <xacro:oak_d_pro_w_camera name="camera" parent_link="base_link">
     <origin xyz="0.40 0.0 0.10" rpy="0 0 0" />
-  </xacro:oak_d_camera>
-  <!-- <xacro:include filename="$(find rover_description)/urdf/xacro/oakd.xacro"/>
-  <xacro:include filename="$(find rover_description)/urdf/xacro/oakd_pro.xacro"/> -->
-  <!-- <xacro:oakd_module parent_link="base_link"/> -->
-  <!-- <xacro:oakd_pro_module parent_link="base_link"/> -->
+  </xacro:oak_d_pro_w_camera> -->
+  <xacro:include filename="$(find rover_description)/urdf/xacro/macros/ouster_os1_lidar_assembly.xacro"/>
+  <xacro:ouster_os1_lidar name="lidar" parent_link="base_link">
+    <origin xyz="0.40 0.0 0.10" rpy="0 0 0" />
+  </xacro:ouster_os1_lidar>
 </robot>

File: src/rover_description/urdf/xacro/macros/sensors.xacro (robot description, xacro)
@@ -1,5 +1,6 @@
 <?xml version="1.0"?>
 <robot xmlns:xacro="http://ros.org/wiki/xacro">
-   <xacro:macro name="camera_sensor"
+# camera sensor macro
+  <xacro:macro name="camera_sensor"
                 params="name parent
                 camera_topic camera_info_topic type:='camera'
@@ -10,6 +11,6 @@
                 clip_near:=0.100 clip_far:=100.0
                 noise_type:='gaussian' noise_mean:=0.0 noise_stddev:=0.0
-                frame_id"
-   >
+                frame_id
+  ">
     <gazebo reference="${parent}">
       <sensor name="${name}" type="${type}">
@@ -40,21 +41,75 @@
     </gazebo>
   </xacro:macro>
-<xacro:macro name="imu_sensor"
-             params="name parent
-             imu_topic
-             fps:=30
-             frame_id
-             ">
-  <gazebo reference="${parent}">
-    <sensor name="${name}" type="imu">
-      <always_on>true</always_on>
-      <visualize>false</visualize>
-      <update_rate>${fps}</update_rate>
-      <topic>${imu_topic}</topic>
-      <imu>
+# imu sensor macro
+  <xacro:macro name="imu_sensor"
+              params="name parent
+              imu_topic
+              fps:=30
+              frame_id
+  ">
+    <gazebo reference="${parent}">
+      <sensor name="${name}" type="imu">
+        <always_on>true</always_on>
+        <visualize>false</visualize>
+        <update_rate>${fps}</update_rate>
+        <topic>${imu_topic}</topic>
+        <imu>
+          <frame_id>${frame_id}</frame_id>
+        </imu>
+      </sensor>
+    </gazebo>
+  </xacro:macro>
+# lidar sensor macro
+  <xacro:macro name="lidar_sensor"
+              params="name parent
+              lidar_topic
+              fps:=30
+              horizontal_samples:=640
+              horizontal_resolution:=1.0
+              horizontal_min_angle:=-1.396263 horizontal_max_angle:=1.396263
+              vertical_samples:=32
+              vertical_resolution:=1.0
+              vertical_min_angle:=-0.5353 vertical_max_angle:=0.1862
+              range_resolution:=0.1
+              range_min:=0.1 range_max:=100.0
+              noise_type:='gaussian' noise_mean:=0.0 noise_stddev:=0.0
+              frame_id
+  ">
+    <gazebo reference="${parent}">
+      <sensor name="${name}" type="gpu_lidar">
+        <always_on>true</always_on>
+        <visualize>false</visualize>
+        <update_rate>${fps}</update_rate>
+        <topic>${lidar_topic}</topic>
+        <gz_frame_id>${frame_id}</gz_frame_id>
+        <lidar>
+          <scan>
+            <horizontal>
+              <samples>${horizontal_samples}</samples>
+              <resolution>${horizontal_resolution}</resolution>
+              <min_angle>${horizontal_min_angle}</min_angle>
+              <max_angle>${horizontal_max_angle}</max_angle>
+            </horizontal>
+            <vertical>
+              <samples>${vertical_samples}</samples>
+              <resolution>${vertical_resolution}</resolution>
+              <min_angle>${vertical_min_angle}</min_angle>
+              <max_angle>${vertical_max_angle}</max_angle>
+            </vertical>
+          </scan>
+          <range>
+            <resolution>${range_resolution}</resolution>
+            <min>${range_min}</min>
+            <max>${range_max}</max>
+          </range>
+          <noise>
+            <type>${noise_type}</type>
+            <mean>${noise_mean}</mean>
+            <stddev>${noise_stddev}</stddev>
+        </noise>
         <frame_id>${frame_id}</frame_id>
-      </imu>
-    </sensor>
-  </gazebo>
-</xacro:macro>
+        </lidar>
+      </sensor>
+    </gazebo>
+  </xacro:macro>
 </robot>

Commit message: feat: integrate Hivision camera and refactor sensor assemblies

File: src/rover_description/urdf/rex.urdf.xacro (robot description, xacro)
@@ -17,7 +17,11 @@
     <origin xyz="0.40 0.0 0.10" rpy="0 0 0" />
   </xacro:oak_d_pro_w_camera> -->
-  <xacro:include filename="$(find rover_description)/urdf/xacro/macros/ouster_os1_lidar_assembly.xacro"/>
+  <!-- <xacro:include filename="$(find rover_description)/urdf/xacro/macros/ouster_os1_lidar_assembly.xacro"/>
   <xacro:ouster_os1_lidar name="lidar" parent_link="base_link">
     <origin xyz="0.40 0.0 0.10" rpy="0 0 0" />
-  </xacro:ouster_os1_lidar>
+  </xacro:ouster_os1_lidar> -->
+  <!-- <xacro:include filename="$(find rover_description)/urdf/xacro/macros/hivision_camera_assembly.xacro"/>
+  <xacro:hivision_camera name="camera" parent_link="base_link">
+    <origin xyz="0.40 0.0 0.10" rpy="0 0 0" />
+  </xacro:hivision_camera> -->
 </robot>
