Commit message: refactor: reorganize urdf structure

File: src/rover_description/urdf/macros/assembly/camera/example_camera_assembly.xacro (robot description, xacro)
@@ -1,5 +1,5 @@
 <?xml version="1.0"?>
 <robot xmlns:xacro="http://www.ros.org/wiki/xacro">
-    <xacro:include filename="$(find rover_description)/urdf/xacro/macros/sensors.xacro"/>
+    <xacro:include filename="$(find rover_description)/urdf/macros/base/sensors.xacro"/>
     <xacro:property name="camera_mesh"       value="package://rover_description/meshes/oak_d_pro_w.dae"/>
     <xacro:property name="camera_mesh_scale" value="0.001 0.001 0.001"/>

File: src/rover_description/urdf/macros/assembly/camera/hivision_camera_assembly.xacro (robot description, xacro)
@@ -1,5 +1,5 @@
 <?xml version="1.0"?>
 <robot xmlns:xacro="http://ros.org/wiki/xacro">
-  <xacro:include filename="$(find rover_description)/urdf/xacro/macros/sensors.xacro"/>
+  <xacro:include filename="$(find rover_description)/urdf/macros/base/sensors.xacro"/>
   <xacro:macro name="hivision_camera" params="name parent_link *origin">
     <xacro:property name="cam_length" value="0.0496"/>

File: src/rover_description/urdf/macros/assembly/camera/oak_d_camera_assembly.xacro (robot description, xacro)
@@ -1,5 +1,5 @@
 <?xml version="1.0"?>
 <robot xmlns:xacro="http://ros.org/wiki/xacro">
-  <xacro:include filename="$(find rover_description)/urdf/xacro/macros/sensors.xacro"/>
+  <xacro:include filename="$(find rover_description)/urdf/macros/base/sensors.xacro"/>
   <xacro:macro name="oak_d_camera" params="name parent_link *origin">
     <xacro:property name="mesh_path"  value="$(find rover_description)/meshes/oak_d.dae"/>
@@ -9,10 +9,10 @@
     <xacro:property name="left_offset"  value="0  0.375 0"/>
     <xacro:property name="right_offset" value="0 -0.375 0"/>
-    <joint name="${name}_center_joint" type="fixed">
+    <joint name="${name}_joint" type="fixed">
       <xacro:insert_block name="origin" />
       <parent link="${parent_link}" />
-      <child  link="${name}_center_link" />
+      <child  link="${name}_link" />
     </joint>
-    <link name="${name}_center_link">
+    <link name="${name}_link">
       <visual>
         <origin xyz="${camera_mesh_xyz}" rpy="${camera_mesh_rpy}" />
@@ -33,5 +33,5 @@
       </inertial>
     </link>
-    <gazebo reference="${name}_center_link">
+    <gazebo reference="${name}_link">
       <visual>
         <material>
@@ -48,37 +48,55 @@
       </visual>
     </gazebo>
-    <joint name="${name}_rgb_optical_joint" type="fixed">
+    <joint name="${name}_rgb_camera_joint" type="fixed">
+      <origin xyz="${left_offset}" rpy="0 0 0" />
+      <parent link="${name}_link" />
+      <child link="${name}_rgb_camera_frame" />
+    </joint>
+    <link name="${name}_rgb_camera_frame"/>
+    <joint name="${name}_rgb_camera_optical_joint" type="fixed">
       <origin xyz="0 0 0" rpy="0 0 0" />
-      <parent link="${name}_center_link" />
-      <child link="${name}_rgb_optical_frame" />
+      <parent link="${name}_rgb_camera_frame" />
+      <child link="${name}_rgb_camera_optical_frame" />
     </joint>
-    <link name="${name}_rgb_optical_frame"/>
+    <link name="${name}_rgb_camera_optical_frame"/>
     <joint name="${name}_left_joint" type="fixed">
       <origin xyz="${left_offset}" rpy="0 0 0" />
-      <parent link="${name}_center_link" />
-      <child link="${name}_left_link" />
+      <parent link="${name}_link" />
+      <child link="${name}_left_camera_frame" />
     </joint>
-    <link name="${name}_left_link"/>
-    <joint name="${name}_left_optical_joint" type="fixed">
+    <link name="${name}_left_camera_frame"/>
+    <joint name="${name}_left_camera_optical_joint" type="fixed">
       <origin xyz="0 0 0" rpy="0 0 0" />
-      <parent link="${name}_left_link" />
-      <child link="${name}_left_optical_frame" />
+      <parent link="${name}_left_camera_frame" />
+      <child link="${name}_left_camera_optical_frame" />
     </joint>
-    <link name="${name}_left_optical_frame"/>
+    <link name="${name}_left_camera_optical_frame"/>
     <joint name="${name}_right_joint" type="fixed">
       <origin xyz="${right_offset}" rpy="0 0 0" />
-      <parent link="${name}_center_link" />
-      <child link="${name}_right_link" />
+      <parent link="${name}_link" />
+      <child link="${name}_right_camera_frame" />
     </joint>
-    <link name="${name}_right_link"/>
-    <joint name="${name}_right_optical_joint" type="fixed">
+    <link name="${name}_right_camera_frame"/>
+    <joint name="${name}_right_camera_optical_joint" type="fixed">
       <origin xyz="0 0 0" rpy="0 0 0" />
-      <parent link="${name}_right_link" />
-      <child link="${name}_right_optical_frame" />
+      <parent link="${name}_right_camera_frame" />
+      <child link="${name}_right_camera_optical_frame" />
     </joint>
-    <link name="${name}_right_optical_frame"/>
+    <link name="${name}_right_camera_optical_frame"/>
+    <joint name="${name}_imu_joint" type="fixed">
+      <origin xyz="0 0 0" rpy="0 0 0" />
+      <parent link="${name}_link" />
+      <child link="${name}_imu_frame" />
+    </joint>
+    <link name="${name}_imu_frame"/>
+    <joint name="${name}_model_joint" type="fixed">
+      <origin xyz="0 0 0" rpy="0 0 0" />
+      <parent link="${name}_link" />
+      <child link="${name}_model_origin" />
+    </joint>
+    <link name="${name}_model_origin"/>
     <xacro:camera_sensor
         name="${name}_rgbd_sensor"
-        parent="${name}_center_link"
+        parent="${name}_rgb_camera_frame"
         camera_topic="${name}/rgbd"
         camera_info_topic="${name}/rgbd/camera_info"
@@ -90,9 +108,9 @@
         clip_near="0.080" clip_far="100.0"
         noise_type="gaussian" noise_mean="0.0" noise_stddev="0.0"
-        frame_id="${name}_rgb_optical_frame"
+        frame_id="${name}_rgb_camera_optical_frame"
         />
     <xacro:camera_sensor
         name="${name}_left_sensor"
-        parent="${name}_left_link"
+        parent="${name}_left_camera_frame"
         camera_topic="${name}/left/image_raw"
         camera_info_topic="${name}/left/camera_info"
@@ -104,9 +122,9 @@
         clip_near="0.196" clip_far="12.0"
         noise_type="gaussian" noise_mean="0.0" noise_stddev="0.0"
-        frame_id="${name}_left_optical_frame"
+        frame_id="${name}_left_camera_optical_frame"
         />
     <xacro:camera_sensor
         name="${name}_right_sensor"
-        parent="${name}_right_link"
+        parent="${name}_right_camera_frame"
         camera_topic="${name}/right/image_raw"
         camera_info_topic="${name}/right/camera_info"
@@ -118,12 +136,12 @@
         clip_near="0.196" clip_far="12.0"
         noise_type="gaussian" noise_mean="0.0" noise_stddev="0.0"
-        frame_id="${name}_right_optical_frame"
+        frame_id="${name}_right_camera_optical_frame"
         />
     <xacro:imu_sensor
         name="${name}_imu"
-        parent="${name}_center_link"
+        parent="${name}_link"
         imu_topic="${name}/imu"
         fps="50.0"
-        frame_id="${name}_center_link"
+        frame_id="${name}_imu_frame"
         />
   </xacro:macro>

File: src/rover_description/urdf/macros/assembly/camera/oak_d_pro_camera_assembly.xacro (robot description, xacro)
@@ -1,7 +1,7 @@
 <?xml version="1.0"?>
 <robot xmlns:xacro="http://ros.org/wiki/xacro">
-  <xacro:include filename="$(find rover_description)/urdf/xacro/macros/sensors.xacro"/>
-  <xacro:macro name="oak_d_pro_w_camera" params="name parent_link *origin">
-    <xacro:property name="mesh_path"  value="$(find rover_description)/meshes/oak_d_pro_w.dae"/>
+  <xacro:include filename="$(find rover_description)/urdf/macros/base/sensors.xacro"/>
+  <xacro:macro name="oak_d_pro_camera" params="name parent_link *origin">
+    <xacro:property name="mesh_path"  value="$(find rover_description)/meshes/oak_d_pro.dae"/>
     <xacro:property name="mesh_scale" value="0.001 0.001 0.001"/>
     <xacro:property name="camera_mesh_xyz" value="-0.022 0.048 -0.00"/>
@@ -9,10 +9,10 @@
     <xacro:property name="left_offset"  value="0  0.375 0"/>
     <xacro:property name="right_offset" value="0 -0.375 0"/>
-    <joint name="${name}_center_joint" type="fixed">
+    <joint name="${name}_joint" type="fixed">
       <xacro:insert_block name="origin" />
       <parent link="${parent_link}" />
-      <child  link="${name}_center_link" />
+      <child  link="${name}_link" />
     </joint>
-    <link name="${name}_center_link">
+    <link name="${name}_link">
       <visual>
         <origin xyz="${camera_mesh_xyz}" rpy="${camera_mesh_rpy}" />
@@ -33,5 +33,5 @@
       </inertial>
     </link>
-    <gazebo reference="${name}_center_link">
+    <gazebo reference="${name}_link">
       <visual>
         <material>
@@ -48,82 +48,100 @@
       </visual>
     </gazebo>
-    <joint name="${name}_rgb_optical_joint" type="fixed">
+    <joint name="${name}_rgb_camera_joint" type="fixed">
+      <origin xyz="${left_offset}" rpy="0 0 0" />
+      <parent link="${name}_link" />
+      <child link="${name}_rgb_camera_frame" />
+    </joint>
+    <link name="${name}_rgb_camera_frame"/>
+    <joint name="${name}_rgb_camera_optical_joint" type="fixed">
       <origin xyz="0 0 0" rpy="0 0 0" />
-      <parent link="${name}_center_link" />
-      <child link="${name}_rgb_optical_frame" />
+      <parent link="${name}_rgb_camera_frame" />
+      <child link="${name}_rgb_camera_optical_frame" />
     </joint>
-    <link name="${name}_rgb_optical_frame"/>
+    <link name="${name}_rgb_camera_optical_frame"/>
     <joint name="${name}_left_joint" type="fixed">
       <origin xyz="${left_offset}" rpy="0 0 0" />
-      <parent link="${name}_center_link" />
-      <child link="${name}_left_link" />
+      <parent link="${name}_link" />
+      <child link="${name}_left_camera_frame" />
     </joint>
-    <link name="${name}_left_link"/>
-    <joint name="${name}_left_optical_joint" type="fixed">
+    <link name="${name}_left_camera_frame"/>
+    <joint name="${name}_left_camera_optical_joint" type="fixed">
       <origin xyz="0 0 0" rpy="0 0 0" />
-      <parent link="${name}_left_link" />
-      <child link="${name}_left_optical_frame" />
+      <parent link="${name}_left_camera_frame" />
+      <child link="${name}_left_camera_optical_frame" />
     </joint>
-    <link name="${name}_left_optical_frame"/>
+    <link name="${name}_left_camera_optical_frame"/>
     <joint name="${name}_right_joint" type="fixed">
       <origin xyz="${right_offset}" rpy="0 0 0" />
-      <parent link="${name}_center_link" />
-      <child link="${name}_right_link" />
+      <parent link="${name}_link" />
+      <child link="${name}_right_camera_frame" />
     </joint>
-    <link name="${name}_right_link"/>
-    <joint name="${name}_right_optical_joint" type="fixed">
+    <link name="${name}_right_camera_frame"/>
+    <joint name="${name}_right_camera_optical_joint" type="fixed">
       <origin xyz="0 0 0" rpy="0 0 0" />
-      <parent link="${name}_right_link" />
-      <child link="${name}_right_optical_frame" />
+      <parent link="${name}_right_camera_frame" />
+      <child link="${name}_right_camera_optical_frame" />
     </joint>
-    <link name="${name}_right_optical_frame"/>
+    <link name="${name}_right_camera_optical_frame"/>
+    <joint name="${name}_imu_joint" type="fixed">
+      <origin xyz="0 0 0" rpy="0 0 0" />
+      <parent link="${name}_link" />
+      <child link="${name}_imu_frame" />
+    </joint>
+    <link name="${name}_imu_frame"/>
+    <joint name="${name}_model_joint" type="fixed">
+      <origin xyz="0 0 0" rpy="0 0 0" />
+      <parent link="${name}_link" />
+      <child link="${name}_model_origin" />
+    </joint>
+    <link name="${name}_model_origin"/>
     <xacro:camera_sensor
-        name="${name}_rgbd_sensor"
-        parent="${name}_center_link"
+      name="${name}_rgbd_sensor"
+      parent="${name}_rgb_camera_frame"
         camera_topic="${name}/rgbd"
         camera_info_topic="${name}/rgbd/camera_info"
         type="rgbd_camera"
         fps="20.0"
-        h_fov="2.21657"
+        h_fov="1.39626"
         width="1280" height="800"
         format="RGB_INT8"
         clip_near="0.10" clip_far="12.0"
         noise_type="gaussian" noise_mean="0.0" noise_stddev="0.0"
-        frame_id="${name}_rgb_optical_frame"
+        frame_id="${name}_rgb_camera_optical_frame"
         />
     <xacro:camera_sensor
         name="${name}_left_sensor"
-        parent="${name}_left_link"
+        parent="${name}_left_camera_frame"
         camera_topic="${name}/left/image_raw"
         camera_info_topic="${name}/left/camera_info"
         type="camera"
         fps="20.0"
-        h_fov="2.21657"
+        h_fov="1.39626"
         width="1280" height="800"
         format="L8"
         clip_near="0.2" clip_far="35.0"
         noise_type="gaussian" noise_mean="0.0" noise_stddev="0.0"
-        frame_id="${name}_left_optical_frame"
+        frame_id="${name}_left_camera_optical_frame"
         />
     <xacro:camera_sensor
         name="${name}_right_sensor"
-        parent="${name}_right_link"
+        parent="${name}_right_camera_frame"
         camera_topic="${name}/right/image_raw"
         camera_info_topic="${name}/right/camera_info"
         type="camera"
         fps="20.0"
-        h_fov="2.21657"
+        h_fov="1.39626"
         width="1280" height="800"
         format="L8"
         clip_near="0.2" clip_far="35.0"
         noise_type="gaussian" noise_mean="0.0" noise_stddev="0.0"
-        frame_id="${name}_right_optical_frame"
+        frame_id="${name}_right_camera_optical_frame"
         />
     <xacro:imu_sensor
         name="${name}_imu"
-        parent="${name}_center_link"
+        parent="${name}_link"
         imu_topic="${name}/imu"
         fps="50.0"
-        frame_id="${name}_center_link"
+        frame_id="${name}_imu_frame"
         />
   </xacro:macro>

File: src/rover_description/urdf/macros/assembly/camera/oak_d_pro_w_camera_assembly.xacro (robot description, xacro)
@@ -1,7 +1,7 @@
 <?xml version="1.0"?>
 <robot xmlns:xacro="http://ros.org/wiki/xacro">
-  <xacro:include filename="$(find rover_description)/urdf/xacro/macros/sensors.xacro"/>
-  <xacro:macro name="oak_d_pro_camera" params="name parent_link *origin">
-    <xacro:property name="mesh_path"  value="$(find rover_description)/meshes/oak_d_pro.dae"/>
+  <xacro:include filename="$(find rover_description)/urdf/macros/base/sensors.xacro"/>
+  <xacro:macro name="oak_d_pro_w_camera" params="name parent_link *origin">
+    <xacro:property name="mesh_path"  value="$(find rover_description)/meshes/oak_d_pro_w.dae"/>
     <xacro:property name="mesh_scale" value="0.001 0.001 0.001"/>
     <xacro:property name="camera_mesh_xyz" value="-0.022 0.048 -0.00"/>
@@ -9,10 +9,10 @@
     <xacro:property name="left_offset"  value="0  0.375 0"/>
     <xacro:property name="right_offset" value="0 -0.375 0"/>
-    <joint name="${name}_center_joint" type="fixed">
+    <joint name="${name}_joint" type="fixed">
       <xacro:insert_block name="origin" />
       <parent link="${parent_link}" />
-      <child  link="${name}_center_link" />
+      <child  link="${name}_link" />
     </joint>
-    <link name="${name}_center_link">
+    <link name="${name}_link">
       <visual>
         <origin xyz="${camera_mesh_xyz}" rpy="${camera_mesh_rpy}" />
@@ -33,5 +33,5 @@
       </inertial>
     </link>
-    <gazebo reference="${name}_center_link">
+    <gazebo reference="${name}_link">
       <visual>
         <material>
@@ -48,82 +48,100 @@
       </visual>
     </gazebo>
-    <joint name="${name}_rgb_optical_joint" type="fixed">
+    <joint name="${name}_rgb_camera_joint" type="fixed">
+      <origin xyz="${left_offset}" rpy="0 0 0" />
+      <parent link="${name}_link" />
+      <child link="${name}_rgb_camera_frame" />
+    </joint>
+    <link name="${name}_rgb_camera_frame"/>
+    <joint name="${name}_rgb_camera_optical_joint" type="fixed">
       <origin xyz="0 0 0" rpy="0 0 0" />
-      <parent link="${name}_center_link" />
-      <child link="${name}_rgb_optical_frame" />
+      <parent link="${name}_rgb_camera_frame" />
+      <child link="${name}_rgb_camera_optical_frame" />
     </joint>
-    <link name="${name}_rgb_optical_frame"/>
+    <link name="${name}_rgb_camera_optical_frame"/>
     <joint name="${name}_left_joint" type="fixed">
       <origin xyz="${left_offset}" rpy="0 0 0" />
-      <parent link="${name}_center_link" />
-      <child link="${name}_left_link" />
+      <parent link="${name}_link" />
+      <child link="${name}_left_camera_frame" />
     </joint>
-    <link name="${name}_left_link"/>
-    <joint name="${name}_left_optical_joint" type="fixed">
+    <link name="${name}_left_camera_frame"/>
+    <joint name="${name}_left_camera_optical_joint" type="fixed">
       <origin xyz="0 0 0" rpy="0 0 0" />
-      <parent link="${name}_left_link" />
-      <child link="${name}_left_optical_frame" />
+      <parent link="${name}_left_camera_frame" />
+      <child link="${name}_left_camera_optical_frame" />
     </joint>
-    <link name="${name}_left_optical_frame"/>
+    <link name="${name}_left_camera_optical_frame"/>
     <joint name="${name}_right_joint" type="fixed">
       <origin xyz="${right_offset}" rpy="0 0 0" />
-      <parent link="${name}_center_link" />
-      <child link="${name}_right_link" />
+      <parent link="${name}_link" />
+      <child link="${name}_right_camera_frame" />
     </joint>
-    <link name="${name}_right_link"/>
-    <joint name="${name}_right_optical_joint" type="fixed">
+    <link name="${name}_right_camera_frame"/>
+    <joint name="${name}_right_camera_optical_joint" type="fixed">
       <origin xyz="0 0 0" rpy="0 0 0" />
-      <parent link="${name}_right_link" />
-      <child link="${name}_right_optical_frame" />
+      <parent link="${name}_right_camera_frame" />
+      <child link="${name}_right_camera_optical_frame" />
     </joint>
-    <link name="${name}_right_optical_frame"/>
+    <link name="${name}_right_camera_optical_frame"/>
+    <joint name="${name}_imu_joint" type="fixed">
+      <origin xyz="0 0 0" rpy="0 0 0" />
+      <parent link="${name}_link" />
+      <child link="${name}_imu_frame" />
+    </joint>
+    <link name="${name}_imu_frame"/>
+    <joint name="${name}_model_joint" type="fixed">
+      <origin xyz="0 0 0" rpy="0 0 0" />
+      <parent link="${name}_link" />
+      <child link="${name}_model_origin" />
+    </joint>
+    <link name="${name}_model_origin"/>
     <xacro:camera_sensor
         name="${name}_rgbd_sensor"
-        parent="${name}_center_link"
+        parent="${name}_rgb_camera_frame"
         camera_topic="${name}/rgbd"
         camera_info_topic="${name}/rgbd/camera_info"
         type="rgbd_camera"
         fps="20.0"
-        h_fov="1.39626"
+        h_fov="2.21657"
         width="1280" height="800"
         format="RGB_INT8"
         clip_near="0.10" clip_far="12.0"
         noise_type="gaussian" noise_mean="0.0" noise_stddev="0.0"
-        frame_id="${name}_rgb_optical_frame"
+        frame_id="${name}_rgb_camera_optical_frame"
         />
     <xacro:camera_sensor
         name="${name}_left_sensor"
-        parent="${name}_left_link"
+        parent="${name}_left_camera_frame"
         camera_topic="${name}/left/image_raw"
         camera_info_topic="${name}/left/camera_info"
         type="camera"
         fps="20.0"
-        h_fov="1.39626"
+        h_fov="2.21657"
         width="1280" height="800"
         format="L8"
         clip_near="0.2" clip_far="35.0"
         noise_type="gaussian" noise_mean="0.0" noise_stddev="0.0"
-        frame_id="${name}_left_optical_frame"
+        frame_id="${name}_left_camera_optical_frame"
         />
     <xacro:camera_sensor
         name="${name}_right_sensor"
-        parent="${name}_right_link"
+        parent="${name}_right_camera_frame"
         camera_topic="${name}/right/image_raw"
         camera_info_topic="${name}/right/camera_info"
         type="camera"
         fps="20.0"
-        h_fov="1.39626"
+        h_fov="2.21657"
         width="1280" height="800"
         format="L8"
         clip_near="0.2" clip_far="35.0"
         noise_type="gaussian" noise_mean="0.0" noise_stddev="0.0"
-        frame_id="${name}_right_optical_frame"
+        frame_id="${name}_right_camera_optical_frame"
         />
     <xacro:imu_sensor
         name="${name}_imu"
-        parent="${name}_center_link"
+        parent="${name}_link"
         imu_topic="${name}/imu"
         fps="50.0"
-        frame_id="${name}_center_link"
+        frame_id="${name}_imu_frame"
         />
   </xacro:macro>

File: src/rover_description/urdf/macros/assembly/lidar/example_lidar_assembly.xacro (robot description, xacro)
@@ -1,5 +1,5 @@
 <?xml version="1.0"?>
 <robot xmlns:xacro="http://www.ros.org/wiki/xacro">
-    <xacro:include filename="$(find rover_description)/urdf/xacro/macros/sensors.xacro"/>
+    <xacro:include filename="$(find rover_description)/urdf/macros/base/sensors.xacro"/>
     <xacro:property name="lidar_mesh"       value="package://rover_description/meshes/ouster_os1.dae"/>
     <xacro:property name="lidar_mesh_scale" value="1 1 1"/>
