Commit message: refactor: reorganize urdf structure

File: src/rover_description/urdf/macros/assembly/lidar/ouster_os1_lidar_assembly.xacro (robot description, xacro)
@@ -1,5 +1,5 @@
 <?xml version="1.0"?>
 <robot xmlns:xacro="http://www.ros.org/wiki/xacro">
-    <xacro:include filename="$(find rover_description)/urdf/xacro/macros/sensors.xacro"/>
+    <xacro:include filename="$(find rover_description)/urdf/macros/base/sensors.xacro"/>
     <xacro:property name="mesh_path"  value="package://rover_description/meshes/ouster_os1.dae"/>
     <xacro:property name="mesh_scale" value="1 1 1"/>
@@ -7,10 +7,10 @@
     <xacro:property name="lidar_mesh_rpy" value="0 0 1.5708"/>
     <xacro:macro name="ouster_os1_lidar" params="name parent_link *origin">
-        <joint name="${name}_center_joint" type="fixed">
+        <joint name="${name}_joint" type="fixed">
             <xacro:insert_block name="origin" />
             <parent link="${parent_link}" />
-            <child  link="${name}_center_link" />
+            <child  link="${name}_link" />
         </joint>
-        <link name="${name}_center_link">
+        <link name="${name}_link">
             <visual>
                 <origin xyz="${lidar_mesh_xyz}" rpy="${lidar_mesh_rpy}" />
@@ -31,5 +31,5 @@
             </inertial>
         </link>
-        <gazebo reference="${name}_center_link">
+        <gazebo reference="${name}_link">
         <visual>
             <material>
@@ -48,11 +48,17 @@
         <joint name="${name}_lidar_joint" type="fixed">
             <origin xyz="0 0 0" rpy="0 0 0" />
-            <parent link="${name}_center_link" />
-            <child  link="${name}_lidar_link" />
+            <parent link="${name}_link" />
+            <child  link="${name}_lidar_frame" />
         </joint>
-        <link name="${name}_lidar_link"/>
+        <link name="${name}_lidar_frame"/>
+        <joint name="${name}_imu_joint" type="fixed">
+            <origin xyz="0 0 0" rpy="0 0 0" />
+            <parent link="${name}_link" />
+            <child link="${name}_imu_frame" />
+        </joint>
+        <link name="${name}_imu_frame"/>
         <xacro:lidar_sensor
             name="${name}_lidar_sensor"
-            parent="${name}_center_link"
+            parent="${name}_link"
             lidar_topic="${name}"
             fps="10"
@@ -66,12 +72,12 @@
             range_min="0.8" range_max="10.0"
             noise_type="gaussian" noise_mean="0.000" noise_stddev="0.003"
-            frame_id="${name}_lidar_link"
+            frame_id="${name}_lidar_frame"
             />
         <xacro:imu_sensor
             name="${name}_imu"
-            parent="${name}_center_link"
+            parent="${name}_link"
             imu_topic="${name}/imu"
             fps="50.0"
-            frame_id="${name}_center_link"
+            frame_id="${name}_imu_frame"
             />
     </xacro:macro>

File: src/rover_description/urdf/rex.urdf.xacro (robot description, xacro)
@@ -13,14 +13,14 @@
   <!-- Gazebo plugins -->
   <xacro:gazebo_plugins/>
-  <!-- <xacro:include filename="$(find rover_description)/urdf/xacro/macros/oak_d_pro_w_camera_assembly.xacro"/>
-  <xacro:oak_d_pro_w_camera name="camera" parent_link="base_link">
-    <origin xyz="0.40 0.0 0.10" rpy="0 0 0" />
-  </xacro:oak_d_pro_w_camera> -->
-  <!-- <xacro:include filename="$(find rover_description)/urdf/xacro/macros/ouster_os1_lidar_assembly.xacro"/>
-  <xacro:ouster_os1_lidar name="lidar" parent_link="base_link">
-    <origin xyz="0.40 0.0 0.10" rpy="0 0 0" />
-  </xacro:ouster_os1_lidar> -->
-  <!-- <xacro:include filename="$(find rover_description)/urdf/xacro/macros/hivision_camera_assembly.xacro"/>
-  <xacro:hivision_camera name="camera" parent_link="base_link">
+  <xacro:include filename="$(find rover_description)/urdf/macros/assembly/camera/oak_d_pro_w_camera_assembly.xacro"/>
+  <xacro:oak_d_pro_w_camera name="camera_00" parent_link="base_link">
+    <origin xyz="0.40 0.0 0.05" rpy="0 0 0" />
+  </xacro:oak_d_pro_w_camera>
+  <xacro:include filename="$(find rover_description)/urdf/macros/assembly/lidar/ouster_os1_lidar_assembly.xacro"/>
+  <xacro:ouster_os1_lidar name="lidar_00" parent_link="base_link">
+    <origin xyz="0.40 0.0 0.15" rpy="0 0 0" />
+  </xacro:ouster_os1_lidar>
+  <!-- <xacro:include filename="$(find rover_description)/urdf/macros/assembly/camera/hivision_camera_assembly.xacro"/>
+  <xacro:hivision_camera name="camera_01" parent_link="base_link">
     <origin xyz="0.40 0.0 0.10" rpy="0 0 0" />
   </xacro:hivision_camera> -->
