Commit message: update(description): refresh rover model and sensor assemblies

File: src/rover_description/urdf/macros/assembly/camera/oak_d_pro_w_camera_assembly.xacro (robot description, xacro)
@@ -3,10 +3,10 @@
   <xacro:include filename="$(find rover_description)/urdf/macros/base/sensors.xacro"/>
   <xacro:macro name="oak_d_pro_w_camera" params="name parent_link *origin">
-    <xacro:property name="mesh_path"  value="$(find rover_description)/meshes/oak_d_pro_w.dae"/>
+    <xacro:property name="mesh_path"  value="package://rover_description/meshes/oak_d_pro_w.dae"/>
     <xacro:property name="mesh_scale" value="0.001 0.001 0.001"/>
     <xacro:property name="camera_mesh_xyz" value="-0.022 0.048 -0.00"/>
     <xacro:property name="camera_mesh_rpy" value="1.5708 0 -1.5708"/>
-    <xacro:property name="left_offset"  value="0  0.375 0"/>
-    <xacro:property name="right_offset" value="0 -0.375 0"/>
+    <xacro:property name="left_offset"  value="0  0.0375 0"/>
+    <xacro:property name="right_offset" value="0 -0.0375 0"/>
     <joint name="${name}_joint" type="fixed">
       <xacro:insert_block name="origin" />

File: src/rover_description/urdf/macros/assembly/lidar/ouster_os1_lidar_assembly.xacro (robot description, xacro)
@@ -59,6 +59,6 @@
         <link name="${name}_imu_frame"/>
         <xacro:lidar_sensor
-            name="${name}_lidar_sensor"
-            parent="${name}_link"
+            name="${name}_lidar"
+            parent="${name}_lidar_frame"
             lidar_topic="${name}"
             fps="10"

File: src/rover_description/urdf/macros/base/sensors.xacro (robot description, xacro)
@@ -19,4 +19,5 @@
         <update_rate>${fps}</update_rate>
         <topic>${camera_topic}</topic>
+        <gz_frame_id>${frame_id}</gz_frame_id>
         <camera>
           <horizontal_fov>${h_fov}</horizontal_fov>
@@ -54,4 +55,5 @@
         <update_rate>${fps}</update_rate>
         <topic>${imu_topic}</topic>
+        <gz_frame_id>${frame_id}</gz_frame_id>
         <imu>
           <frame_id>${frame_id}</frame_id>

File: src/rover_description/urdf/rex.urdf.xacro (robot description, xacro)
@@ -23,7 +23,7 @@
     <origin xyz="0.40 0.0 0.15" rpy="0 0 0" />
   </xacro:ouster_os1_lidar> -->
-  <xacro:include filename="$(find rover_description)/urdf/macros/assembly/camera/hivision_camera_assembly.xacro"/>
+  <!-- <xacro:include filename="$(find rover_description)/urdf/macros/assembly/camera/hivision_camera_assembly.xacro"/>
   <xacro:hivision_camera name="camera_xx" parent_link="base_link">
     <origin xyz="0.40 0.0 0.10" rpy="0 0 0" />
-  </xacro:hivision_camera>
+  </xacro:hivision_camera> -->
 </robot>

File: src/rover_description/urdf/xacro/autonomy_submodule.xacro (robot description, xacro)
@@ -9,8 +9,8 @@
             </inertial>
         </link>
-        <joint name="mount_link_joint" type="revolute">
+        <joint name="mount_link_joint" type="fixed">
             <parent link="${parent_link}"/>
             <child link="mount_link"/>
-            <origin xyz="-0.27 0.0 0.0" rpy="0 0 0"/>
+            <origin xyz="0.27 0.0 0.0" rpy="0 0 3.14159265359"/>
             <axis xyz="0 0 1"/>
             <limit effort="5" velocity="1.0" lower="-3.14" upper="3.14"/>
@@ -23,5 +23,5 @@
             </inertial>
         </link>
-        <joint name="sensor_mount_00_joint" type="revolute">
+        <joint name="sensor_mount_00_joint" type="fixed">
             <parent link="mount_link"/>
             <child link="sensor_mount_00_link"/>
@@ -37,5 +37,5 @@
             </inertial>
         </link>
-        <joint name="sensor_mount_01_joint" type="revolute">
+        <joint name="sensor_mount_01_joint" type="fixed">
             <parent link="mount_link"/>
             <child link="sensor_mount_01_link"/>

File: src/rover_description/urdf/xacro/base.xacro (robot description, xacro)
@@ -1,4 +1,5 @@
 <?xml version="1.0"?>
 <robot xmlns:xacro="http://www.ros.org/wiki/xacro">
+  <xacro:include filename="$(find rover_description)/urdf/macros/base/inertial.xacro"/>
   <!-- Main body -->
   <xacro:macro name="base_link">
@@ -19,12 +20,11 @@
         </geometry>
       </collision>
-      <inertial>
+      <xacro:inertial_box mass="15" x="0.7" y="0.44" z="0.176">
         <origin xyz="0 0 0" rpy="0 0 0"/>
-        <mass value="15"/>
-        <inertia ixx="0.28072" ixy="0" ixz="0"
-                              iyy="0.65122" iyz="0"
-                                            izz="0.8545"/>
-      </inertial>
+      </xacro:inertial_box>
     </link>
+    <gazebo reference="base_link">
+      <selfCollide>true</selfCollide>
+    </gazebo>
   </xacro:macro>
 </robot>

File: src/rover_description/urdf/xacro/gazebo_plugins.xacro (robot description, xacro)
@@ -29,11 +29,11 @@
         <jointA>base_link_to_swivel_right</jointA>
         <jointB>base_link_to_swivel_left</jointB>
-        <forceConstant>100.0</forceConstant>
+        <forceConstant>60.0</forceConstant>
         <bogieJoint>arm_pivot_left_to_arm_front_left</bogieJoint>
         <bogieJoint>arm_pivot_left_to_arm_rear_left</bogieJoint>
         <bogieJoint>arm_pivot_right_to_arm_front_right</bogieJoint>
         <bogieJoint>arm_pivot_right_to_arm_rear_right</bogieJoint>
-        <bogieSpring>200.0</bogieSpring>
-        <bogieDamping>20.0</bogieDamping>
+        <bogieSpring>100.0</bogieSpring>
+        <bogieDamping>10.0</bogieDamping>
       </plugin>
       <!-- ===== Steering controllers (position) ===== -->
@@ -56,6 +56,6 @@
       <use_velocity_commands>true</use_velocity_commands>
       <joint_index>0</joint_index>
-      <cmd_max> 0.65</cmd_max>
-      <cmd_min>-0.65</cmd_min>
+      <cmd_max> 1.5</cmd_max>
+      <cmd_min>-1.5</cmd_min>
     </plugin>
   </xacro:macro>
@@ -67,9 +67,9 @@
       <initial_velocity>0.0</initial_velocity>
       <use_force_commands>true</use_force_commands>
-      <p_gain>0.5</p_gain>
-      <i_gain>0.5</i_gain>
+      <p_gain>0.45</p_gain>
+      <i_gain>0.35</i_gain>
       <d_gain>0.0001</d_gain>
-      <cmd_max> 50.0</cmd_max>
-      <cmd_min>-50.0</cmd_min>
+      <cmd_max> 45.0</cmd_max>
+      <cmd_min>-45.0</cmd_min>
     </plugin>
   </xacro:macro>

File: src/rover_description/urdf/xacro/wheel_assembly.xacro (robot description, xacro)
@@ -1,4 +1,5 @@
 <?xml version="1.0"?>
 <robot xmlns:xacro="http://www.ros.org/wiki/xacro">
+  <xacro:include filename="$(find rover_description)/urdf/macros/base/inertial.xacro"/>
   <!-- Single wheel -->
   <xacro:macro name="wheel_assembly" params="name parent x">
@@ -28,11 +29,7 @@
         </geometry>
       </collision>
-      <inertial>
-        <origin xyz="0 0 0" rpy="0 0 0"/>
-        <mass value="0.001"/>
-        <inertia ixx="0.000001" ixy="0" ixz="0"
-                               iyy="0.000001" iyz="0"
-                                              izz="0.000001"/>
-      </inertial>
+      <xacro:inertial_cylinder mass="0.001" length="0.05" radius="0.025">
+        <origin xyz="0 0 0" rpy="0 0 0"/>
+      </xacro:inertial_cylinder>
     </link>
     <!-- Drive joint -->
@@ -60,19 +57,33 @@
         </geometry>
       </collision>
-      <inertial>
-        <mass value="3"/>
-        <inertia ixx="0.015025" ixy="0" ixz="0"
-                               iyy="0.015025" iyz="0"
-                                              izz="0.0216"/>
-      </inertial>
+      <xacro:inertial_cylinder mass="3" length="0.13" radius="0.125">
+        <origin xyz="0 0 0" rpy="0 0 0"/>
+      </xacro:inertial_cylinder>
     </link>
     <!-- Wheel ground contact properties -->
     <gazebo reference="wheel_${name}">
-      <mu>1.5</mu>
-      <mu2>1.5</mu2>
-      <slip1>0.00062</slip1>
-      <slip2>0.0</slip2>
-      <fdir1>1 0 0</fdir1>
-      <maxContacts>10</maxContacts>
+      <surface>
+        <friction>
+          <ode>
+            <mu>1.5</mu>
+            <mu2>1.5</mu2>
+            <slip1>0.00062</slip1>
+            <slip2>0.0</slip2>
+          </ode>
+          <bullet>
+            <friction>1.5</friction>
+            <friction2>1.5</friction2>
+          </bullet>
+        </friction>
+        <contact>
+          <ode>
+            <max_contacts>10</max_contacts>
+          </ode>
+          <bullet>
+            <soft_cfm>0.001</soft_cfm>
+            <soft_erp>0.2</soft_erp>
+          </bullet>
+        </contact>
+      </surface>
     </gazebo>
   </xacro:macro>
@@ -84,7 +95,10 @@
       <origin xyz="0 ${base_y} 0" rpy="0 0 0"/>
       <axis xyz="0 1 0"/>
-      <limit effort="1000.0" lower="-1" upper="1" velocity="0.5"/>
+      <limit effort="1000.0" lower="-1.15" upper="1.15" velocity="0.6"/>
       <dynamics friction="1.0" damping="0.1"/>
     </joint>
+    <gazebo reference="swivel_${side}">
+      <selfCollide>true</selfCollide>
+    </gazebo>
     <!-- Swivel pin -->
     <link name="swivel_${side}">
@@ -104,11 +118,7 @@
         </geometry>
       </collision>
-      <inertial>
-        <origin xyz="0 0 0" rpy="0 0 0"/>
-        <mass value="0.001"/>
-        <inertia ixx="0.000001" ixy="0" ixz="0"
-                               iyy="0.000001" iyz="0"
-                                              izz="0.000001"/>
-      </inertial>
+      <xacro:inertial_cylinder mass="0.001" length="0.107" radius="0.01">
+        <origin xyz="0 0 0" rpy="0 0 0"/>
+      </xacro:inertial_cylinder>
     </link>
     <!-- Fixed connection: swivel to center -->
@@ -135,12 +145,11 @@
         </geometry>
       </collision>
-      <inertial>
-        <origin xyz="0 0 0" rpy="0 0 0"/>
-        <mass value="0.3"/>
-        <inertia ixx="0.000213" ixy="0" ixz="0"
-                               iyy="0.000340" iyz="0"
-                                              izz="0.000373"/>
-      </inertial>
-    </link>
+      <xacro:inertial_box mass="0.3" x="0.10" y="0.07" z="0.06">
+        <origin xyz="0 0 0" rpy="0 0 0"/>
+      </xacro:inertial_box>
+    </link>
+    <gazebo reference="arm_pivot_${side}">
+      <selfCollide>true</selfCollide>
+    </gazebo>
     <!-- Front arm half -->
     <joint name="arm_pivot_${side}_to_arm_front_${side}" type="revolute">
@@ -149,6 +158,6 @@
       <origin xyz="0.05 0 0" rpy="0 0 0"/>
       <axis xyz="0 1 0"/>
-      <limit effort="500.0" lower="-0.5" upper="0.5" velocity="0.5"/>
-      <dynamics friction="0.5" damping="0.1"/>
+      <limit effort="500.0" lower="-0.7" upper="0.7" velocity="0.6"/>
+      <dynamics friction="0.3" damping="0.05"/>
     </joint>
     <!-- Front arm beam -->
@@ -169,12 +178,11 @@
         </geometry>
       </collision>
-      <inertial>
+      <xacro:inertial_box mass="0.4" x="0.45" y="0.04" z="0.04">
         <origin xyz="0.225 0 0" rpy="0 0 0"/>
-        <mass value="0.4"/>
-        <inertia ixx="0.000107" ixy="0" ixz="0"
-                               iyy="0.006803" iyz="0"
-                                              izz="0.006803"/>
-      </inertial>
-    </link>
+      </xacro:inertial_box>
+    </link>
+    <gazebo reference="arm_front_${side}">
+      <selfCollide>true</selfCollide>
+    </gazebo>
     <!-- Rear arm half -->
     <joint name="arm_pivot_${side}_to_arm_rear_${side}" type="revolute">
@@ -183,6 +191,6 @@
       <origin xyz="-0.05 0 0" rpy="0 0 0"/>
       <axis xyz="0 1 0"/>
-      <limit effort="500.0" lower="-0.5" upper="0.5" velocity="0.5"/>
-      <dynamics friction="0.5" damping="0.1"/>
+      <limit effort="500.0" lower="-0.7" upper="0.7" velocity="0.6"/>
+      <dynamics friction="0.3" damping="0.05"/>
     </joint>
     <!-- Rear arm beam -->
@@ -203,13 +211,11 @@
         </geometry>
       </collision>
-      <inertial>
+      <xacro:inertial_box mass="0.4" x="0.45" y="0.04" z="0.04">
         <origin xyz="-0.225 0 0" rpy="0 0 0"/>
-        <mass value="0.4"/>
-        <inertia ixx="0.000107"
-                 ixy="0" ixz="0"
-                 iyy="0.006803" iyz="0"
-                 izz="0.006803"/>
-      </inertial>
-    </link>
+      </xacro:inertial_box>
+    </link>
+    <gazebo reference="arm_rear_${side}">
+      <selfCollide>true</selfCollide>
+    </gazebo>
     <!-- Wheels -->
     <xacro:wheel_assembly name="front_${side}" parent="arm_front_${side}" x="0.40"/>
